Commit message: update for super_lio

File: src/gld_robot_description/model/my_description.urdf (robot description, URDF)
Before this commit: robot gld_robot_description, 3 links, 2 joints
Links:
- removed link chassis
Joints:
- removed joint base_to_chassis
- removed joint chassis_to_livox_frame
- added joint imu_to_livox: type fixed, parent base_footprint, child livox_frame, origin xyz=0.0 0.0 0.0 rpy=3.1416 0.0 -1.5708
